File: pcb/Macropad.kicad_pcb (KiCad board)
At the start: 2 copper layers, 50.5 x 84 mm, 17 parts, among them SW1 CherryMX, SW2 CherryMX, SW3 CherryMX, SW5 CherryMX, U2 KY-040, U3 MOUDLE-SEEEDUINO-XIAO-ESP32C3

Commit message: update
Parts:
- removed R4, R5: 500, Resistor_SMD:R_0805_2012Metric
Routing:
- net GND: track 72.2 -> 65.5 mm
- net Net-(U3-PA5_A9_D9_MISO): track 65.0 -> 58.8 mm
- net Net-(U3-PA6_A10_D10_MOSI): track 92.5 -> 87.5 mm
