File: pcb/Macropad.kicad_sch (KiCad schematic)
At the start: 17 parts, among them SW1 CherryMX, SW2 CherryMX, SW3 CherryMX, SW5 CherryMX, U2 KY-040, U3 MOUDLE-SEEEDUINO-XIAO-ESP32C3

Commit message: update
Parts:
- removed R4, R5: 500, Resistor_SMD:R_0805_2012Metric, symbol Device:R
